Commit message: first commit

File: urdf/husky.urdf.xacro (robot description, xacro)
@@ -228,31 +228,4 @@
     </joint>
   </transmission>
-  <joint name="scan_joint" type="fixed">
-    <parent link="base_link"/>
-    <child link="base_scan"/>
-    <origin xyz="0.2 0 0.25" rpy="0 0 0"/>
-  </joint>
-  <link name="base_scan">
-    <visual>
-      <origin xyz="0.2 0 0.25" rpy="0 0 0"/>
-      <geometry>
-        <mesh filename="package://igvc_world/meshes/sensors/lds.stl" scale="0.001 0.001 0.001"/>
-      </geometry>
-      <material name="dark"/>
-    </visual>
-    <collision>
-      <origin xyz="0.2 0 0.25" rpy="0 0 0"/>
-      <geometry>
-        <cylinder length="0.0315" radius="0.055"/>
-      </geometry>
-    </collision>
-    <inertial>
-      <mass value="0.114" />
-      <origin xyz="0 0 0" />
-      <inertia ixx="0.001" ixy="0.0" ixz="0.0"
-               iyy="0.001" iyz="0.0"
-               izz="0.001" />
-    </inertial>
-  </link>
   <joint name="camera_joint" type="fixed">
     <origin xyz="0 0 1.3" rpy="-1.57 0 -1.57"/>
